File: mtf122.kicad_pcb (KiCad board)
At the start: 2 copper layers, 500 x 194 mm, 216 parts, among them J1 CONN_CAP_IBM_F, SW1 1,8, SW10 A,8, SW100 6,2, SW101 7,2, SW102 7,1, SW103 8,2, SW104 9,1, SW105 A,1, SW106 A,2, SW107 B,2, SW108 C,2, SW109 D,2, SW11 B,8, SW110 D,3, SW111 E,3, SW112 E,2, SW113 F,3, SW114 G,3, SW115 G,2, SW116 1,1, SW117 2,1, SW118 3,1, SW119 4,1, SW12 C,8, SW120 6,1, SW121 8,1, SW122 C,1, SW123 D,1, SW124 E,1, SW125 F,1, SW126 F,2, SW127 G,1, SW13 1,7, SW14 2,7, SW15 3,7, SW16 4,7, SW17 5,7, SW18 6,7, SW19 7,7, SW2 2,8, SW20 8,7, SW21 9,7, SW22 A,7, SW23 B,7, SW24 C,7, SW25 1,5, SW26 1,6, SW27 2,6, SW28 3,6, SW29 4,6, SW3 3,8, SW30 5,6, SW31 5,5, SW32 6,6, SW33 7,6, SW34 8,5, SW35 8,6, SW36 9,6, SW37 9,5, SW38 A,6, SW39 B,6, SW4 4,8, SW40 C,6, SW41 D,7, SW42 D,8, SW43 E,7, SW44 E,8, SW45 F,7, SW46 F,8, SW47 G,7, SW48 G,8, SW49 1,4, SW5 5,8, SW50 2,4, SW51 2,5, SW52 3,5, SW53 4,5, SW54 5,4, SW55 6,5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

Commit message: Cleanup and schematic update
Parts:
- removed C1_TEST, C2_TEST, C3_TEST, C4_TEST, C5_TEST, C6_TEST, C7_TEST, C8_TEST, C9_TEST, CA_TEST, CB_TEST, CC_TEST, CD_TEST, CE_TEST, CF_TEST, CG_TEST, R1_TEST, R2_TEST (x2), R3_TEST, R4_TEST, R5_TEST, R6_TEST, R8_TEST: TestPoint_Pad_D1.0mm, TestPoint:TestPoint_Pad_D1.0mm
- removed REF** (x63): HOLE, lib_fp:HOLE
- added COL_1_TP9: C1_TestPoint, TestPoint:TestPoint_Pad_D1.0mm, B.Cu at (61.2, 296.1)
- added COL_2_TP10: C2_TestPoint, TestPoint:TestPoint_Pad_D1.0mm, B.Cu at (88.4, 296.0)
- added COL_3_TP11: C3_TestPoint, TestPoint:TestPoint_Pad_D1.0mm, B.Cu at (121.2, 296.0)
- added COL_4_TP12: C4_TestPoint, TestPoint:TestPoint_Pad_D1.0mm, B.Cu at (160.5, 296.0)
- added COL_5_TP13: C5_TestPoint, TestPoint:TestPoint_Pad_D1.0mm, B.Cu at (178.2, 273.4)
- added COL_6_TP14: C6_TestPoint, TestPoint:TestPoint_Pad_D1.0mm, B.Cu at (241.2, 296.0)
- added COL_7_TP15: C7_TestPoint, TestPoint:TestPoint_Pad_D1.0mm, B.Cu at (245.9, 273.3)
- added COL_8_TP16: C8_TestPoint, TestPoint:TestPoint_Pad_D1.0mm, B.Cu at (321.9, 295.9)
- added COL_9_TP17: C9_TestPoint, TestPoint:TestPoint_Pad_D1.0mm, B.Cu at (283.9, 279.3)
- added COL_A_TP18: CA_TestPoint, TestPoint:TestPoint_Pad_D1.0mm, B.Cu at (321.9, 273.2)
- added COL_B_TP19: CB_TestPoint, TestPoint:TestPoint_Pad_D1.0mm, B.Cu at (351.4, 289.0)
- added COL_C_TP20: CC_TestPoint, TestPoint:TestPoint_Pad_D1.0mm, B.Cu at (377.7, 296.1)
- added COL_D_TP21: CD_TestPoint, TestPoint:TestPoint_Pad_D1.0mm, B.Cu at (421.2, 295.6)
- added COL_E_TP22: CE_TestPoint, TestPoint:TestPoint_Pad_D1.0mm, B.Cu at (468.2, 295.6)
- added COL_F_TP23: CF_TestPoint, TestPoint:TestPoint_Pad_D1.0mm, B.Cu at (506.2, 295.6)
- added COL_G_TP24: CG_TestPoint, TestPoint:TestPoint_Pad_D1.0mm, B.Cu at (533.5, 295.7)
- added H1: HOLE, lib_fp:HOLE, F.Cu at (55.8, 233.3)
- added H10: HOLE, lib_fp:HOLE, F.Cu at (120.3, 149.3)
- added H11: HOLE, lib_fp:HOLE, F.Cu at (120.3, 170.3)
- added H12: HOLE, lib_fp:HOLE, F.Cu at (126.6, 212.3)
- added H13: HOLE, lib_fp:HOLE, F.Cu at (140.8, 191.3)
- added H14: HOLE, lib_fp:HOLE, F.Cu at (145.5, 254.3)
- added H15: HOLE, lib_fp:HOLE, F.Cu at (145.6, 295.4)
- added H16: HOLE, lib_fp:HOLE, F.Cu at (155.0, 275.4)
- added H17: HOLE, lib_fp:HOLE, F.Cu at (169.3, 212.3)
- added H18: HOLE, lib_fp:HOLE, F.Cu at (174.1, 233.3)
- added H19: HOLE, lib_fp:HOLE, F.Cu at (178.8, 128.3)
- added H2: HOLE, lib_fp:HOLE, F.Cu at (55.8, 275.3)
- added H20: HOLE, lib_fp:HOLE, F.Cu at (178.8, 149.3)
- added H21: HOLE, lib_fp:HOLE, F.Cu at (178.8, 170.3)
- added H22: HOLE, lib_fp:HOLE, F.Cu at (216.8, 149.3)
- added H23: HOLE, lib_fp:HOLE, F.Cu at (216.8, 191.3)
- added H24: HOLE, lib_fp:HOLE, F.Cu at (221.6, 254.3)
- added H25: HOLE, lib_fp:HOLE, F.Cu at (221.5, 295.4)
- added H26: HOLE, lib_fp:HOLE, F.Cu at (245.3, 212.3)
- added H27: HOLE, lib_fp:HOLE, F.Cu at (250.0, 233.3)
- added H28: HOLE, lib_fp:HOLE, F.Cu at (254.8, 128.3)
- added H29: HOLE, lib_fp:HOLE, F.Cu at (254.8, 170.3)
- added H3: HOLE, lib_fp:HOLE, F.Cu at (74.8, 191.3)
- added H30: HOLE, lib_fp:HOLE, F.Cu at (254.8, 275.4)
- added H31: HOLE, lib_fp:HOLE, F.Cu at (259.6, 254.3)
- added H32: HOLE, lib_fp:HOLE, F.Cu at (292.8, 128.3)
- added H33: HOLE, lib_fp:HOLE, F.Cu at (292.8, 149.3)
- added H34: HOLE, lib_fp:HOLE, F.Cu at (292.8, 191.3)
- added H35: HOLE, lib_fp:HOLE, F.Cu at (292.8, 295.4)
- added H36: HOLE, lib_fp:HOLE, F.Cu at (313.1, 275.4)
- added H37: HOLE, lib_fp:HOLE, F.Cu at (321.3, 212.3)
- added H38: HOLE, lib_fp:HOLE, F.Cu at (326.1, 233.3)
- added H39: HOLE, lib_fp:HOLE, F.Cu at (330.8, 128.3)
- added H4: HOLE, lib_fp:HOLE, F.Cu at (74.8, 212.3)
- added H40: HOLE, lib_fp:HOLE, F.Cu at (330.8, 170.3)
- added H41: HOLE, lib_fp:HOLE, F.Cu at (335.6, 254.3)
- added H42: HOLE, lib_fp:HOLE, F.Cu at (338.5, 295.4)
- added H43: HOLE, lib_fp:HOLE, F.Cu at (364.0, 275.4)
- added H44: HOLE, lib_fp:HOLE, F.Cu at (368.8, 191.3)
- added H45: HOLE, lib_fp:HOLE, F.Cu at (392.3, 212.3)
- added H46: HOLE, lib_fp:HOLE, F.Cu at (396.8, 233.3)
- added H47: HOLE, lib_fp:HOLE, F.Cu at (396.8, 254.3)
- added H48: HOLE, lib_fp:HOLE, F.Cu at (396.8, 275.3)
- added H49: HOLE, lib_fp:HOLE, F.Cu at (396.8, 295.3)
- added H5: HOLE, lib_fp:HOLE, F.Cu at (74.8, 254.3)
- added H50: HOLE, lib_fp:HOLE, F.Cu at (415.8, 191.3)
- added H51: HOLE, lib_fp:HOLE, F.Cu at (434.8, 233.3)
- added H52: HOLE, lib_fp:HOLE, F.Cu at (434.8, 254.3)
- added H53: HOLE, lib_fp:HOLE, F.Cu at (434.8, 275.3)
- added H54: HOLE, lib_fp:HOLE, F.Cu at (453.8, 191.3)
- added H55: HOLE, lib_fp:HOLE, F.Cu at (453.8, 295.3)
- added H56: HOLE, lib_fp:HOLE, F.Cu at (462.8, 212.3)
- added H57: HOLE, lib_fp:HOLE, F.Cu at (481.8, 233.3)
- added H58: HOLE, lib_fp:HOLE, F.Cu at (481.8, 275.3)
- added H59: HOLE, lib_fp:HOLE, F.Cu at (500.8, 191.3)
- added H6: HOLE, lib_fp:HOLE, F.Cu at (74.8, 295.3)
- added H60: HOLE, lib_fp:HOLE, F.Cu at (538.8, 233.3)
- added H61: HOLE, lib_fp:HOLE, F.Cu at (538.8, 254.3)
- added H62: HOLE, lib_fp:HOLE, F.Cu at (538.8, 275.3)
- added H63: HOLE, lib_fp:HOLE, F.Cu at (538.8, 296.3)
- added H7: HOLE, lib_fp:HOLE, F.Cu at (104.6, 233.3)
- added H8: HOLE, lib_fp:HOLE, F.Cu at (107.6, 275.3)
- added H9: HOLE, lib_fp:HOLE, F.Cu at (120.3, 128.3)
- added ROW_1_TP1: R1_TestPoint, TestPoint:TestPoint_Pad_D1.0mm, F.Cu at (533.8, 275.6)
- added ROW_2_TP2: R2_TestPoint, TestPoint:TestPoint_Pad_D1.0mm, F.Cu at (541.4, 264.8)
- added ROW_3_TP3: R3_TestPoint, TestPoint:TestPoint_Pad_D1.0mm, F.Cu at (533.7, 254.5)
- added ROW_4_TP4: R4_TestPoint, TestPoint:TestPoint_Pad_D1.0mm, F.Cu at (526.5, 253.5)
- added ROW_5_TP5: R5_TestPoint, TestPoint:TestPoint_Pad_D1.0mm, F.Cu at (541.4, 222.8)
- added ROW_6_TP6: R6_TestPoint, TestPoint:TestPoint_Pad_D1.0mm, F.Cu at (533.7, 213.0)
- added ROW_7_TP7: R7_TestPoint, TestPoint:TestPoint_Pad_D1.0mm, F.Cu at (526.5, 212.0)
- added ROW_8_TP8: R8_TestPoint, TestPoint:TestPoint_Pad_D1.0mm, F.Cu at (541.4, 201.8)
