File: mtf122.kicad_pcb (KiCad board)
At the start: 2 copper layers, 500 x 194 mm, 192 parts, among them J1 CONN_CAP_IBM_F, SW1 1,8, SW10 A,8, SW100 6,2, SW101 7,2, SW102 7,1, SW103 8,2, SW104 9,1, SW105 A,1, SW106 A,2, SW107 B,2, SW108 C,2, SW109 D,2, SW11 B,8, SW110 D,3, SW111 E,3, SW112 E,2, SW113 F,3, SW114 G,3, SW115 G,2, SW116 1,1, SW117 2,1, SW118 3,1, SW119 4,1, SW12 C,8, SW120 6,1, SW121 8,1, SW122 C,1, SW123 D,1, SW124 E,1, SW125 F,1, SW126 F,2, SW127 G,1, SW13 1,7, SW14 2,7, SW15 3,7, SW16 4,7, SW17 5,7, SW18 6,7, SW19 7,7, SW2 2,8, SW20 8,7, SW21 9,7, SW22 A,7, SW23 B,7, SW24 C,7, SW25 1,5, SW26 1,6, SW27 2,6, SW28 3,6, SW29 4,6, SW3 3,8, SW30 5,6, SW31 5,5, SW32 6,6, SW33 7,6, SW34 8,5, SW35 8,6, SW36 9,6, SW37 9,5, SW38 A,6, SW39 B,6, SW4 4,8, SW40 C,6, SW41 D,7, SW42 D,8, SW43 E,7, SW44 E,8, SW45 F,7, SW46 F,8, SW47 G,7, SW48 G,8, SW49 1,4, SW5 5,8, SW50 2,4, SW51 2,5, SW52 3,5, SW53 4,5, SW54 5,4, SW55 6,5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

Commit message: Added extra appendages to be compliant with IBM rules
Routing:
- net GND: track 9588.0 -> 9654.9 mm
- net ROW_1: track 882.4 -> 915.3 mm
- net ROW_3: track 850.3 -> 878.3 mm
- net ROW_7: track 661.6 -> 689.5 mm
- net ROW_6: track 751.6 -> 779.6 mm
- net COL_A: track 298.0 -> 313.5 mm
- net COL_7: track 240.4 -> 255.0 mm
- net COL_5: track 208.0 -> 222.6 mm
- net COL_9: track 266.5 -> 280.9 mm
- net ROW_4: track 858.1 -> 867.1 mm

Commit message: Added test points for testing continuity on ROWS
Parts:
- added R1_TEST: TestPoint_Pad_D1.0mm, TestPoint:TestPoint_Pad_D1.0mm, F.Cu at (533.8, 275.6)
- added R2_TEST: TestPoint_Pad_D1.0mm, TestPoint:TestPoint_Pad_D1.0mm, F.Cu at (526.0, 212.0)
- added R2_TEST: TestPoint_Pad_D1.0mm, TestPoint:TestPoint_Pad_D1.0mm, F.Cu at (541.4, 264.8)
- added R3_TEST: TestPoint_Pad_D1.0mm, TestPoint:TestPoint_Pad_D1.0mm, F.Cu at (533.7, 254.5)
- added R4_TEST: TestPoint_Pad_D1.0mm, TestPoint:TestPoint_Pad_D1.0mm, F.Cu at (526.0, 253.5)
- added R5_TEST: TestPoint_Pad_D1.0mm, TestPoint:TestPoint_Pad_D1.0mm, F.Cu at (541.4, 222.8)
- added R6_TEST: TestPoint_Pad_D1.0mm, TestPoint:TestPoint_Pad_D1.0mm, F.Cu at (533.7, 213.0)
- added R8_TEST: TestPoint_Pad_D1.0mm, TestPoint:TestPoint_Pad_D1.0mm, F.Cu at (541.4, 201.8)
Routing:
- net ROW_5: track 796.4 -> 804.1 mm
- net ROW_2: track 898.1 -> 905.8 mm
- net ROW_8: track 686.1 -> 693.7 mm

Commit message: Added test points for testing continuity on COLUMNS
Parts:
- added C1_TEST: TestPoint_Pad_D1.0mm, TestPoint:TestPoint_Pad_D1.0mm, F.Cu at (61.2, 296.1)
- added C2_TEST: TestPoint_Pad_D1.0mm, TestPoint:TestPoint_Pad_D1.0mm, F.Cu at (88.4, 296.0)
- added C3_TEST: TestPoint_Pad_D1.0mm, TestPoint:TestPoint_Pad_D1.0mm, F.Cu at (121.2, 296.0)
- added C4_TEST: TestPoint_Pad_D1.0mm, TestPoint:TestPoint_Pad_D1.0mm, F.Cu at (160.5, 296.0)
- added C5_TEST: TestPoint_Pad_D1.0mm, TestPoint:TestPoint_Pad_D1.0mm, F.Cu at (178.2, 273.4)
- added C6_TEST: TestPoint_Pad_D1.0mm, TestPoint:TestPoint_Pad_D1.0mm, F.Cu at (241.2, 296.0)
- added C7_TEST: TestPoint_Pad_D1.0mm, TestPoint:TestPoint_Pad_D1.0mm, F.Cu at (245.9, 273.3)
- added C8_TEST: TestPoint_Pad_D1.0mm, TestPoint:TestPoint_Pad_D1.0mm, F.Cu at (321.9, 295.9)
- added C9_TEST: TestPoint_Pad_D1.0mm, TestPoint:TestPoint_Pad_D1.0mm, F.Cu at (283.9, 279.3)
- added CA_TEST: TestPoint_Pad_D1.0mm, TestPoint:TestPoint_Pad_D1.0mm, F.Cu at (321.9, 273.2)
- added CB_TEST: TestPoint_Pad_D1.0mm, TestPoint:TestPoint_Pad_D1.0mm, F.Cu at (351.4, 289.1)
- added CC_TEST: TestPoint_Pad_D1.0mm, TestPoint:TestPoint_Pad_D1.0mm, F.Cu at (377.7, 296.1)
- added CD_TEST: TestPoint_Pad_D1.0mm, TestPoint:TestPoint_Pad_D1.0mm, F.Cu at (421.2, 295.6)
- added CE_TEST: TestPoint_Pad_D1.0mm, TestPoint:TestPoint_Pad_D1.0mm, F.Cu at (468.2, 295.6)
- added CF_TEST: TestPoint_Pad_D1.0mm, TestPoint:TestPoint_Pad_D1.0mm, F.Cu at (506.2, 295.6)
- added CG_TEST: TestPoint_Pad_D1.0mm, TestPoint:TestPoint_Pad_D1.0mm, F.Cu at (533.5, 295.7)
Routing:
- net GND: track 9654.9 -> 9744.3 mm
- net COL_6: track 275.5 -> 285.7 mm
- net COL_2: track 240.5 -> 250.7 mm
- net COL_4: track 239.0 -> 249.2 mm
- net COL_3: track 205.4 -> 215.5 mm
- net COL_1: track 257.3 -> 267.5 mm
- net COL_C: track 345.5 -> 355.6 mm
- net COL_8: track 325.0 -> 335.0 mm
- net COL_G: track 493.9 -> 503.7 mm
- net COL_F: track 466.5 -> 476.3 mm
- net COL_E: track 440.9 -> 450.7 mm
- net COL_D: track 397.2 -> 407.0 mm
- net COL_5: track 222.6 -> 231.0 mm
- net COL_7: track 255.0 -> 263.4 mm
- net COL_A: track 313.5 -> 321.8 mm
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
Commit message: 1- Resized the top edge of the PCB to fit inside the keyboard without any permanent irreversable modification. 2- Routed the connections to take less space 3- Added a GND fill zone on the back of the PCB (necessary?) 4- Relocated part of the silk screen graphics and text 5- Incremented the revision of the board to rev.2
Routing:
- net GND: track 9744.3 -> 9467.2 mm
- net COL_1: track 267.5 -> 289.8 mm
- net COL_2: track 250.7 -> 272.4 mm
- net COL_3: track 215.5 -> 233.7 mm
- net ROW_8: track 693.7 -> 702.6 mm
- net ROW_4: track 867.1 -> 875.9 mm
- net ROW_7: track 689.5 -> 697.8 mm
- net COL_D: track 407.0 -> 415.0 mm
- net ROW_3: track 878.3 -> 885.9 mm
- net COL_E: track 450.7 -> 457.2 mm
- net ROW_2: track 905.8 -> 912.2 mm
- net COL_F: track 476.3 -> 482.5 mm
- net COL_G: track 503.7 -> 509.5 mm
- net ROW_1: track 920.0 -> 925.6 mm
- net COL_C: track 355.6 -> 360.8 mm
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- added copper zone on B.Cu, net GND
Other:
- outline, holes or cut-outs redrawn
- board text added: "IBM-M122-CAP Rev. 2 #:"
- board text removed: "IBM-M122-CAP Rev. 1 #:"

Commit message: Removed column test points from F.SilkS
Parts:
- C1_TEST, C2_TEST, C3_TEST, C4_TEST, C5_TEST, C6_TEST, C7_TEST, C8_TEST, C9_TEST, CA_TEST, CB_TEST, CC_TEST, CD_TEST, CE_TEST, CF_TEST, CG_TEST: moved to B.Cu
